File: pcb/orione.kicad_pcb (KiCad board)
At the start: 2 copper layers, 445.6 x 143.8 mm, 192 parts, among them J1 Conn_02x10_Odd_Even, J2 Conn_02x10_Odd_Even

Commit message: minor updtaes to pcb
Parts:
- removed H8: MountingHole_Pad, MountingHole:MountingHole_3.2mm_M3_Pad_Via
- added D89: LED, LED_THT:LED_D5.0mm, F.Cu at (74.8, 123.4)
- added D89: LED, LED_THT:LED_D5.0mm, F.Cu at (74.9, 148.1)
- added J3: Conn_02x03_Odd_Even, Connector_PinHeader_2.54mm:PinHeader_2x03_P2.54mm_Horizontal, F.Cu at (71.5, 104.0)
- added R1: Resistor, Resistor_THT:R_Axial_DIN0207_L6.3mm_D2.5mm_P10.16mm_Horizontal, F.Cu at (78.6, 131.3)
- added R1: Resistor, Resistor_THT:R_Axial_DIN0207_L6.3mm_D2.5mm_P10.16mm_Horizontal, F.Cu at (78.7, 156.0)
- moved H7 66.5 mm to (486.5, 171.0)
- moved D11 35.6 mm to (410.3, 106.9)
- moved D16 35.6 mm to (514.7, 106.8)
- moved D14 35.6 mm to (476.6, 106.8)
- moved D17 35.6 mm to (181.7, 135.4)
- moved D2 35.6 mm to (219.8, 106.8)
- moved D21 35.6 mm to (257.9, 135.4)
- moved D23 35.6 mm to (296.0, 135.4)
- moved D24 35.6 mm to (315.0, 135.4)
- moved D27 35.6 mm to (372.2, 135.4)
- moved D28 35.6 mm to (391.2, 135.4)
- moved D31 35.6 mm to (477.0, 135.4)
- moved D36 35.6 mm to (229.3, 154.4)
- moved D38 35.6 mm to (267.4, 154.4)
- moved D39 35.6 mm to (286.5, 154.4)
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Connections:
- net Net-(J2-Pin_2) renamed GND 0
- J1 pad 3: unconnected-(J1-Pin_3-Pad3) -> Led 1
- J1 pad 4: unconnected-(J1-Pin_4-Pad4) -> GND 1
Routing:
- net GND 1: track 0.00 -> 64.0 mm
- net Led 1: track 0.00 -> 46.7 mm
- net Net-(D89-A): track 0.00 -> 37.4 mm
- net GND 0: track 1049.4 -> 1081.0 mm
- net Column 15: track 523.6 -> 526.9 mm
Other:
- board size 445.6 x 143.8 mm -> 477.1 x 143.8 mm
- board text added: "Caps Lock"
- board text added: "MSP432"
- board text added: "Power"
