File: pcb/orione-v1/orione-v1.kicad_pcb (KiCad board)
At the start: 2 copper layers, 497.9 x 142.8 mm, 192 parts, among them J1 Conn_02x10_Odd_Even, J2 Conn_02x10_Odd_Even, J3 Conn_02x03_Odd_Even, SW1 SW_Push, SW10 SW_Push, SW11 SW_Push, SW12 SW_Push, SW13 SW_Push, SW14 SW_Push, SW15 SW_Push, SW16 SW_Push, SW17 SW_Push, SW18 SW_Push, SW19 SW_Push, SW2 SW_Push, SW20 SW_Push, SW21 SW_Push, SW22 SW_Push, SW23 SW_Push, SW24 SW_Push, SW25 SW_Push, SW26 SW_Push, SW27 SW_Push, SW28 SW_Push, SW29 SW_Push, SW3 SW_Push, SW30 SW_Push, SW31 SW_Push, SW32 SW_Push, SW33 SW_Push, SW34 SW_Push, SW35 SW_Push, SW36 SW_Push, SW37 SW_Push, SW38 SW_Push, SW39 SW_Push, SW4 SW_Push, SW40 SW_Push, SW41 SW_Push, SW42 SW_Push, SW43 SW_Push, SW44 SW_Push, SW45 SW_Push, SW46 SW_Push, SW47 SW_Push, SW48 SW_Push, SW49 SW_Push, SW5 SW_Push, SW50 SW_Push, SW51 SW_Push, SW52 SW_Push, SW53 SW_Push, SW54 SW_Push, SW55 SW_Push, SW56 SW_Push, SW57 SW_Push, SW58 SW_Push, SW59 SW_Push, SW6 SW_Push, SW60 SW_Push, SW61 SW_Push, SW62 SW_Push, SW63 SW_Push, SW64 SW_Push, SW65 SW_Push, SW66 SW_Push, SW67 SW_Push, SW68 SW_Push, SW69 SW_Push, SW7 SW_Push, SW70 SW_Push, SW71 SW_Push, SW72 SW_Push, SW73 SW_Push, SW74 SW_Push, SW75 SW_Push, SW76 SW_Push, SW77 SW_Push, SW78 SW_Push, SW79 SW_Push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

Commit message: pcv v1.1
Parts:
- J3: value Conn_02x03_Odd_Even -> Conn_01x06_Pin; footprint Connector_PinHeader_2.54mm:PinHeader_2x03_P2.54mm_Horizontal -> Connector_PinHeader_2.54mm:PinHeader_1x06_P2.54mm_Horizontal; moved to B.Cu
- moved D89 83.6 mm to (123.0, 178.6)
- moved R1 83.6 mm to (119.4, 186.4)
- moved R2 77.6 mm to (144.0, 186.4)
- moved D90 77.6 mm to (147.8, 178.8)
- moved G*** 74.5 mm to (120.4, 106.0)
- moved J3 56.8 mm to (142.9, 81.9)
- moved H5 24.8 mm to (94.9, 190.1)
- moved H1 24.8 mm to (94.7, 75.8)
Connections:
- H1 pad 1: Net-(J1-Pin_19) -> Net-(D89-K)
- H2 pad 1: Net-(J1-Pin_19) -> Net-(D89-K)
- H3 pad 1: Net-(J1-Pin_19) -> Net-(D89-K)
- H4 pad 1: Net-(J1-Pin_19) -> Net-(D89-K)
- H5 pad 1: Net-(J1-Pin_19) -> Net-(D89-K)
- H6 pad 1: Net-(J1-Pin_19) -> Net-(D89-K)
- H7 pad 1: Net-(J1-Pin_19) -> Net-(D89-K)
- H8 pad 1: Net-(J1-Pin_19) -> Net-(D89-K)
- J1 pad 1: unconnected-(J1-Pin_1-Pad1) -> Net-(J1-Pin_1)
- J1 pad 11: Row 1 -> Net-(J1-Pin_11)
- J1 pad 13: Row 0 -> unconnected-(J1-Pin_13-Pad13)
- J1 pad 19: Net-(J1-Pin_19) -> unconnected-(J1-Pin_19-Pad19)
- J1 pad 3: Row 5 -> unconnected-(J1-Pin_3-Pad3)
- J1 pad 5: Row 4 -> Net-(J1-Pin_5)
- J1 pad 7: Row 3 -> Net-(J1-Pin_7)
- J1 pad 9: Row 2 -> Net-(J1-Pin_9)
- J2 pad 12: unconnected-(J2-Pin_12-Pad12) -> Row 1
- J2 pad 14: unconnected-(J2-Pin_14-Pad14) -> Row 2
- J2 pad 16: unconnected-(J2-Pin_16-Pad16) -> Row 3
- J2 pad 18: unconnected-(J2-Pin_18-Pad18) -> Row 4
- J2 pad 20: unconnected-(J2-Pin_20-Pad20) -> Row 5
- J2 pad 6: unconnected-(J2-Pin_6-Pad6) -> Net-(J2-Pin_6)
- J2 pad 8: unconnected-(J2-Pin_8-Pad8) -> Row 0
- J3 pad 1: unconnected-(J3-Pin_1-Pad1) -> Net-(J2-Pin_2)
- J3 pad 2: unconnected-(J3-Pin_2-Pad2) -> Net-(J1-Pin_11)
- J3 pad 3: unconnected-(J3-Pin_3-Pad3) -> Net-(J1-Pin_1)
- J3 pad 4: unconnected-(J3-Pin_4-Pad4) -> Net-(J1-Pin_7)
- J3 pad 5: unconnected-(J3-Pin_5-Pad5) -> Net-(J1-Pin_5)
- J3 pad 6: unconnected-(J3-Pin_6-Pad6) -> Net-(J1-Pin_9)
- R1 pad 2: Net-(J2-Pin_4) -> Net-(J2-Pin_6)
- R2 pad 2: Net-(J2-Pin_2) -> Net-(J2-Pin_4)
Routing:
- net Net-(J1-Pin_19): track 978.9 -> 0.00 mm, vias 1 -> 0
- net Net-(D89-K): track 69.1 -> 1028.0 mm, vias 0 -> 1
- net Net-(J2-Pin_6): track 0.00 -> 93.1 mm
- net Net-(J1-Pin_11): track 0.00 -> 77.2 mm
- net Row 4: track 441.5 -> 371.0 mm
- net Row 2: track 457.7 -> 387.6 mm
- net Row 5: track 471.7 -> 404.1 mm
- net Row 1: track 454.2 -> 386.6 mm
- net Row 3: track 359.0 -> 292.7 mm
- net Net-(J1-Pin_9): track 0.00 -> 60.8 mm
- net Net-(J1-Pin_7): track 0.00 -> 59.2 mm
- net Row 0: track 462.5 -> 404.7 mm
- net Net-(J1-Pin_5): track 0.00 -> 56.4 mm
- net Net-(J1-Pin_1): track 0.00 -> 50.4 mm
- net Net-(J2-Pin_2): track 86.6 -> 47.5 mm, vias 1 -> 0
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Other:
- board size 497.9 x 142.8 mm -> 473.1 x 142.8 mm
- board text added: "CTS"
- board text added: "GND"
- board text added: "RTS"
- board text added: "RXD"
- board text added: "TXD"
- board text added: "VCC"

Commit message: fixed GND
Connections:
- D89 pad 1: Net-(D89-K) -> GND
- D90 pad 1: Net-(D89-K) -> GND
- H1 pad 1: Net-(D89-K) -> GND
- H2 pad 1: Net-(D89-K) -> GND
- H3 pad 1: Net-(D89-K) -> GND
- H4 pad 1: Net-(D89-K) -> GND
- H5 pad 1: Net-(D89-K) -> GND
- H6 pad 1: Net-(D89-K) -> GND
- H7 pad 1: Net-(D89-K) -> GND
- H8 pad 1: Net-(D89-K) -> GND
- J1 pad 4: Net-(D89-K) -> GND
- J2 pad 2: Net-(J2-Pin_2) -> GND
- J3 pad 1: Net-(J2-Pin_2) -> GND
Routing:
- net Net-(D89-K): track 1028.0 -> 0.00 mm, vias 1 -> 0
- net Net-(J2-Pin_2): track 47.5 -> 0.00 mm
- net GND: track 0.00 -> 8.37 mm, vias 0 -> 1
- net Net-(J2-Pin_6): track 93.1 -> 91.0 mm
- net Net-(J2-Pin_4): track 82.2 -> 80.1 mm
- net Column 15: track 507.3 -> 508.0 mm
- added copper zone on B.Cu, net GND
- added copper zone on F.Cu, net GND
