File: pcb/orione-v1/orione-v1.kicad_pcb (KiCad board)
At the start: 2 copper layers, 473.1 x 142.8 mm, 192 parts, among them J1 Conn_02x10_Odd_Even, J2 Conn_02x10_Odd_Even, J3 Conn_01x06_Pin, SW1 SW_Push, SW10 SW_Push, SW11 SW_Push, SW12 SW_Push, SW13 SW_Push, SW14 SW_Push, SW15 SW_Push, SW16 SW_Push, SW17 SW_Push, SW18 SW_Push, SW19 SW_Push, SW2 SW_Push, SW20 SW_Push, SW21 SW_Push, SW22 SW_Push, SW23 SW_Push, SW24 SW_Push, SW25 SW_Push, SW26 SW_Push, SW27 SW_Push, SW28 SW_Push, SW29 SW_Push, SW3 SW_Push, SW30 SW_Push, SW31 SW_Push, SW32 SW_Push, SW33 SW_Push, SW34 SW_Push, SW35 SW_Push, SW36 SW_Push, SW37 SW_Push, SW38 SW_Push, SW39 SW_Push, SW4 SW_Push, SW40 SW_Push, SW41 SW_Push, SW42 SW_Push, SW43 SW_Push, SW44 SW_Push, SW45 SW_Push, SW46 SW_Push, SW47 SW_Push, SW48 SW_Push, SW49 SW_Push, SW5 SW_Push, SW50 SW_Push, SW51 SW_Push, SW52 SW_Push, SW53 SW_Push, SW54 SW_Push, SW55 SW_Push, SW56 SW_Push, SW57 SW_Push, SW58 SW_Push, SW59 SW_Push, SW6 SW_Push, SW60 SW_Push, SW61 SW_Push, SW62 SW_Push, SW63 SW_Push, SW64 SW_Push, SW65 SW_Push, SW66 SW_Push, SW67 SW_Push, SW68 SW_Push, SW69 SW_Push, SW7 SW_Push, SW70 SW_Push, SW71 SW_Push, SW72 SW_Push, SW73 SW_Push, SW74 SW_Push, SW75 SW_Push, SW76 SW_Push, SW77 SW_Push, SW78 SW_Push, SW79 SW_Push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

Commit message: added voltage divider
Parts:
- added R3: R, Resistor_THT:R_Axial_DIN0207_L6.3mm_D2.5mm_P10.16mm_Horizontal, F.Cu at (149.9, 81.8)
- added R4: R, Resistor_THT:R_Axial_DIN0207_L6.3mm_D2.5mm_P10.16mm_Horizontal, F.Cu at (156.9, 81.8)
Connections:
- J3 pad 3: Net-(J1-Pin_1) -> Net-(J3-Pin_3)
Routing:
- net Net-(J3-Pin_3): track 0.00 -> 15.2 mm
- net Net-(J1-Pin_1): track 50.4 -> 55.6 mm

Commit message: changed pin layout of uart
Connections:
- J1 pad 11: Net-(J1-Pin_11) -> unconnected-(J1-Pin_11-Pad11)
- J1 pad 3: unconnected-(J1-Pin_3-Pad3) -> Net-(J1-Pin_3)
- J3 pad 2: Net-(J1-Pin_11) -> Net-(J1-Pin_3)
Routing:
- net Net-(J1-Pin_11): track 77.2 -> 0.00 mm
- net Net-(J1-Pin_3): track 0.00 -> 56.1 mm
Changed lines of the file:
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@@
 	(net 110 "Net-(J1-Pin_7)")
 	(net 111 "Column 11")
-	(net 112 "Net-(J1-Pin_11)")
+	(net 112 "unconnected-(J1-Pin_11-Pad11)")
 	(net 113 "Column 13")
 	(net 114 "GND")
@@
 	(net 126 "Net-(D90-A)")
 	(net 127 "Net-(J1-Pin_1)")
-	(net 128 "unconnected-(J1-Pin_3-Pad3)")
+	(net 128 "Net-(J1-Pin_3)")
 	(net 129 "unconnected-(J1-Pin_2-Pad2)")
 	(net 130 "Net-(J3-Pin_3)")
@@
 			(layers "*.Cu" "*.Mask")
 			(remove_unused_layers no)
-			(net 128 "unconnected-(J1-Pin_3-Pad3)")
+			(net 128 "Net-(J1-Pin_3)")
 			(pinfunction "Pin_3")
-			(pintype "passive+no_connect")
+			(pintype "passive")
 		)
 		(pad "4" thru_hole oval
@@
 			(layers "*.Cu" "*.Mask")
 			(remove_unused_layers no)
-			(net 112 "Net-(J1-Pin_11)")
+			(net 112 "unconnected-(J1-Pin_11-Pad11)")
 			(pinfunction "Pin_11")
-			(pintype "passive")
+			(pintype "passive+no_connect")
 		)
 		(pad "12" thru_hole oval
@@
 			(layers "*.Cu" "*.Mask")
 			(remove_unused_layers no)
-			(net 112 "Net-(J1-Pin_11)")
+			(net 128 "Net-(J1-Pin_3)")
 			(pinfunction "Pin_2")
 			(pintype "passive")
@@
 	)
 	(segment
-		(start 130.17375 81.86384)
-		(end 109.88375 102.15384)
+		(start 109.86375 102.17384)
+		(end 109.86375 128.53884)
 		(width 0.2)
 		(layer "B.Cu")
@@
 	)
 	(segment
-		(start 109.88375 128.55884)
-		(end 113.89375 132.56884)
+		(start 130.17375 81.86384)
+		(end 109.86375 102.17384)
 		(width 0.2)
 		(layer "B.Cu")
@@
 	)
 	(segment
-		(start 109.88375 102.15384)
-		(end 109.88375 128.55884)
+		(start 109.86375 128.53884)
+		(end 113.89375 132.56884)
 		(width 0.2)
 		(layer "B.Cu")
@@
 	)
 	(segment
-		(start 111.30375 105.81384)
-		(end 135.25375 81.86384)
+		(start 113.89375 130.02884)
+		(end 111.01375 127.14884)
 		(width 0.2)
 		(layer "F.Cu")
@@
 	)
 	(segment
-		(start 111.30375 127.43884)
-		(end 111.30375 105.81384)
+		(start 111.01375 106.10384)
+		(end 135.25375 81.86384)
 		(width 0.2)
 		(layer "F.Cu")
@@
 	)
 	(segment
-		(start 113.89375 130.02884)
-		(end 111.30375 127.43884)
+		(start 111.01375 127.14884)
+		(end 111.01375 106.10384)
 		(width 0.2)
 		(layer "F.Cu")
@@
 	)
 	(segment
-		(start 137.69375 79.22384)
-		(end 130.69375 79.22384)
-		(width 0.2)
-		(layer "F.Cu")
-		(net 112)
-	)
-	(segment
-		(start 140.33375 81.86384)
-		(end 137.69375 79.22384)
-		(width 0.2)
-		(layer "F.Cu")
-		(net 112)
-	)
-	(segment
-		(start 109.48375 100.43384)
-		(end 109.48375 130.69884)
-		(width 0.2)
-		(layer "F.Cu")
-		(net 112)
-	)
-	(segment
-		(start 109.48375 130.69884)
-		(end 113.89375 135.10884)
-		(width 0.2)
-		(layer "F.Cu")
-		(net 112)
-	)
-	(segment
-		(start 130.69375 79.22384)
-		(end 109.48375 100.43384)
-		(width 0.2)
-		(layer "F.Cu")
-		(net 112)
-	)
-	(segment
 		(start 441.01 168.83134)
 		(end 455.2975 183.11884)
@@
 	)
 	(segment
-		(start 110.28375 123.87884)
-		(end 110.28375 104.29384)
+		(start 113.89375 127.48884)
+		(end 110.26375 123.85884)
 		(width 0.2)
 		(layer "B.Cu")
@@
 	)
 	(segment
-		(start 113.89375 127.48884)
-		(end 110.28375 123.87884)
+		(start 110.26375 123.85884)
+		(end 110.26375 104.31384)
 		(width 0.2)
 		(layer "B.Cu")
@@
 	)
 	(segment
-		(start 110.28375 104.29384)
+		(start 110.26375 104.31384)
 		(end 132.71375 81.86384)
 		(width 0.2)
@@
 	)
 	(segment
+		(start 111.41375 110.78384)
+		(end 111.41375 122.46884)
+		(width 0.2)
+		(layer "F.Cu")
+		(net 128)
+	)
+	(segment
+		(start 140.33375 81.86384)
+		(end 111.41375 110.78384)
+		(width 0.2)
+		(layer "F.Cu")
+		(net 128)
+	)
+	(segment
+		(start 111.41375 122.46884)
+		(end 113.89375 124.94884)
+		(width 0.2)
+		(layer "F.Cu")
+		(net 128)
+	)
+	(segment
 		(start 116.46875 122.40884)
 		(end 116.43375 122.40884)
@@
 		(polygon
 			(pts
-				(xy 72.47375 57.28384) (xy 72.47375 209.21384) (xy 561.20375 209.21384) (xy 561.59375 55.73384)
+				(xy 71.24375 55.92384) (xy 71.24375 214.73384) (xy 558.64375 215.30384) (xy 561.53375 52.45384)
 			)
 		)

Commit message: modified pcb based on new parts
Parts:
- removed R3, R4: R, Resistor_THT:R_Axial_DIN0207_L6.3mm_D2.5mm_P10.16mm_Horizontal
- added U1: LD1117_TO220, Package_TO_SOT_THT:TO-220-3_Vertical, F.Cu at (175.8, 85.6)
Connections:
- J1 pad 3: Net-(J1-Pin_3) -> unconnected-(J1-Pin_3-Pad3)
- J1 pad 9: Net-(J1-Pin_9) -> unconnected-(J1-Pin_9-Pad9)
- J3 pad 2: Net-(J1-Pin_3) -> unconnected-(J3-Pin_2-Pad2)
- J3 pad 6: Net-(J1-Pin_9) -> unconnected-(J3-Pin_6-Pad6)
Routing:
- net Net-(J1-Pin_9): track 60.8 -> 0.00 mm
- net Net-(J1-Pin_3): track 56.1 -> 0.00 mm
- net Net-(J3-Pin_3): track 15.2 -> 39.5 mm
- net Net-(J1-Pin_1): track 55.6 -> 75.0 mm
