File: pcb/orione-v1/orione-v1.kicad_pcb (KiCad board)
At the start: 2 copper layers, 473.1 x 142.8 mm, 193 parts, among them J1 Conn_02x10_Odd_Even, J2 Conn_02x10_Odd_Even, J3 Conn_01x06_Pin, SW1 SW_Push, SW10 SW_Push, SW11 SW_Push, SW12 SW_Push, SW13 SW_Push, SW14 SW_Push, SW15 SW_Push, SW16 SW_Push, SW17 SW_Push, SW18 SW_Push, SW19 SW_Push, SW2 SW_Push, SW20 SW_Push, SW21 SW_Push, SW22 SW_Push, SW23 SW_Push, SW24 SW_Push, SW25 SW_Push, SW26 SW_Push, SW27 SW_Push, SW28 SW_Push, SW29 SW_Push, SW3 SW_Push, SW30 SW_Push, SW31 SW_Push, SW32 SW_Push, SW33 SW_Push, SW34 SW_Push, SW35 SW_Push, SW36 SW_Push, SW37 SW_Push, SW38 SW_Push, SW39 SW_Push, SW4 SW_Push, SW40 SW_Push, SW41 SW_Push, SW42 SW_Push, SW43 SW_Push, SW44 SW_Push, SW45 SW_Push, SW46 SW_Push, SW47 SW_Push, SW48 SW_Push, SW49 SW_Push, SW5 SW_Push, SW50 SW_Push, SW51 SW_Push, SW52 SW_Push, SW53 SW_Push, SW54 SW_Push, SW55 SW_Push, SW56 SW_Push, SW57 SW_Push, SW58 SW_Push, SW59 SW_Push, SW6 SW_Push, SW60 SW_Push, SW61 SW_Push, SW62 SW_Push, SW63 SW_Push, SW64 SW_Push, SW65 SW_Push, SW66 SW_Push, SW67 SW_Push, SW68 SW_Push, SW69 SW_Push, SW7 SW_Push, SW70 SW_Push, SW71 SW_Push, SW72 SW_Push, SW73 SW_Push, SW74 SW_Push, SW75 SW_Push, SW76 SW_Push, SW77 SW_Push, SW78 SW_Push, SW79 SW_Push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

Commit message: added to pcb rotary encoder and oled dysplay
Parts:
- added J4: Conn_01x04_Socket, Connector_PinSocket_2.54mm:PinSocket_1x04_P2.54mm_Vertical, F.Cu at (509.2, 55.3)
- added SW89: RotaryEncoder_Switch_MP, Rotary_Encoder:RotaryEncoder_Bourns_Vertical_PEC12R-3x17F-Sxxxx, F.Cu at (521.3, 56.7)
Connections:
- J1 pad 11: unconnected-(J1-Pin_11-Pad11) -> Net-(J1-Pin_11)
- J1 pad 13: unconnected-(J1-Pin_13-Pad13) -> Net-(J1-Pin_13)
- J1 pad 15: unconnected-(J1-Pin_15-Pad15) -> Net-(J1-Pin_15)
- J1 pad 17: unconnected-(J1-Pin_17-Pad17) -> Net-(J1-Pin_17)
- J1 pad 19: unconnected-(J1-Pin_19-Pad19) -> Net-(J1-Pin_19)
- J1 pad 9: unconnected-(J1-Pin_9-Pad9) -> Net-(J1-Pin_9)
Routing:
- net Net-(J1-Pin_13): track 0.00 -> 507.0 mm
- net Net-(J1-Pin_15): track 0.00 -> 504.6 mm
- net Net-(J1-Pin_11): track 0.00 -> 476.8 mm
- net Net-(J1-Pin_19): track 0.00 -> 473.0 mm
- net Net-(J1-Pin_17): track 0.00 -> 472.4 mm, vias 0 -> 1
- net Net-(J1-Pin_9): track 0.00 -> 471.5 mm
- net Net-(J1-Pin_1): track 75.0 -> 507.2 mm
- net GND: vias 1 -> 2
Other:
- board size 473.1 x 142.8 mm -> 473.1 x 161.4 mm

Commit message: prova
Parts:
- removed H1, H2, H3, H4, H5, H6, H7, H8: MountingHole_Pad, MountingHole:MountingHole_3.2mm_M3_Pad_Via
- removed J4: Conn_01x04_Socket, Connector_PinSocket_2.54mm:PinSocket_1x04_P2.54mm_Vertical
- removed SW89: RotaryEncoder_Switch_MP, Rotary_Encoder:RotaryEncoder_Bourns_Vertical_PEC12R-3x17F-Sxxxx
- removed U1: LD1117_TO220, Package_TO_SOT_THT:TO-220-3_Vertical
- added C1: C_Polarized, Capacitor_THT:CP_Radial_Tantal_D4.5mm_P5.00mm, F.Cu at (279.3, -66.0)
- added C2: C_Polarized, Capacitor_THT:CP_Radial_Tantal_D4.5mm_P5.00mm, F.Cu at (279.3, -57.5)
- added C3: C, Capacitor_THT:C_Radial_D10.0mm_H12.5mm_P5.00mm, F.Cu at (269.3, -64.4)
- added C4: C, Capacitor_THT:C_Radial_D10.0mm_H12.5mm_P5.00mm, F.Cu at (269.3, -52.9)
- added C5: C, Capacitor_THT:C_Radial_D10.0mm_H12.5mm_P5.00mm, F.Cu at (269.3, -41.3)
- added C6: C, Capacitor_THT:C_Radial_D10.0mm_H12.5mm_P5.00mm, F.Cu at (269.3, -29.8)
- added SW90: RotaryEncoder, Rotary_Encoder:RotaryEncoder_Alps_EC12E_Vertical_H20mm, F.Cu at (279.3, -48.1)
- added U2: TLV1117-50, Package_TO_SOT_THT:TO-220-3_Vertical, F.Cu at (280.8, -34.0)
- D1, D10, D11, D12, D13, D14, D15, D16, D17, D18, D19, D2, D20, D21, D22, D23, D24, D25, D26, D27, D28, D29, D3, D30, D31, D32, D33, D34, D35, D36, D37, D38, D39, D4, D40, D41, D42, D43, D44, D45, D46, D47, D48, D49, D5, D50, D51, D52, D53, D54, D55, D56, D57, D58, D59, D6, D60, D61, D62, D63, D64, D65, D66, D67, D68, D69, D7, D70, D71, D72, D73, D74, D75, D76, D77, D78, D79, D8, D80, D81, D82, D83, D84, D85, D86, D87, D88, D9: footprint Resistor_THT:R_Axial_DIN0207_L6.3mm_D2.5mm_P10.16mm_Horizontal -> Resistor_THT:R_Axial_DIN0204_L3.6mm_D1.6mm_P5.08mm_Horizontal; moved to F.Cu
- moved D16 366.2 mm to (171.8, 72.4), turned to 0 degrees
- moved D15 347.0 mm to (171.8, 75.6), turned to 0 degrees
- moved D14 327.9 mm to (171.8, 78.7), turned to 0 degrees
- moved D13 299.3 mm to (171.8, 81.9), turned to 0 degrees
- moved D33 293.4 mm to (252.3, 46.2), turned to -90 degrees
- moved D12 280.2 mm to (171.8, 85.0), turned to 0 degrees
- moved D32 278.0 mm to (249.2, 46.2), turned to -90 degrees
- moved D31 262.6 mm to (246.0, 46.2), turned to -90 degrees
- moved D11 261.1 mm to (171.8, 88.2), turned to 0 degrees
- moved D10 242.1 mm to (171.8, 91.3), turned to 0 degrees
- moved D79 238.7 mm to (432.0, 59.0), turned to -90 degrees
- moved D30 238.2 mm to (242.9, 46.2), turned to -90 degrees
- moved D50 230.4 mm to (323.7, 48.3), turned to -90 degrees
- moved D80 221.8 mm to (435.2, 59.0), turned to -90 degrees
- moved D49 215.7 mm to (320.5, 48.3), turned to -90 degrees
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Connections:
- J1 pad 13: Net-(J1-Pin_13) -> unconnected-(J1-Pin_13-Pad13)
- J1 pad 15: Net-(J1-Pin_15) -> unconnected-(J1-Pin_15-Pad15)
- J1 pad 17: Net-(J1-Pin_17) -> unconnected-(J1-Pin_17-Pad17)
- J1 pad 19: Net-(J1-Pin_19) -> unconnected-(J1-Pin_19-Pad19)
Routing:
- net Net-(J1-Pin_1): track 507.2 -> 0.00 mm
- net Net-(J1-Pin_13): track 507.0 -> 0.00 mm
- net Net-(J1-Pin_15): track 504.6 -> 0.00 mm
- net Net-(J1-Pin_11): track 476.8 -> 0.00 mm
- net Net-(J1-Pin_19): track 473.0 -> 0.00 mm
- net Net-(J1-Pin_17): track 472.4 -> 0.00 mm, vias 1 -> 0
- net Net-(J1-Pin_9): track 471.5 -> 0.00 mm
- net Column 16: track 528.5 -> 104.8 mm, vias 1 -> 0
- net Row 0: track 404.7 -> 0.00 mm
- net Column 15: track 508.0 -> 107.3 mm, vias 1 -> 0
- net Row 5: track 404.1 -> 31.5 mm
- net Column 14: track 476.0 -> 104.8 mm, vias 1 -> 0
- net Row 2: track 387.6 -> 51.1 mm
- net Row 1: track 386.6 -> 50.4 mm
- net Row 4: track 371.0 -> 48.1 mm
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- removed copper zone on B.Cu, net GND
- removed copper zone on F.Cu, net GND
Other:
- board outline removed
- board text removed: "Orione v1"

Commit message: wip
Parts:
- moved SW90 267.2 mm to (523.9, 59.7)
- moved D85 259.1 mm to (192.5, 40.0)
- moved D84 242.6 mm to (206.3, 35.5)
- moved D86 241.7 mm to (215.4, 21.0)
- moved D83 230.7 mm to (215.2, 35.0)
- moved D79 215.7 mm to (216.3, 56.9)
- moved D82 213.2 mm to (229.4, 37.3)
- moved D87 209.5 mm to (248.6, 40.0)
- moved D88 209.5 mm to (251.7, 40.0)
- moved D80 197.7 mm to (237.4, 56.9)
- moved D8 183.5 mm to (350.7, 56.9), turned to -90 degrees
- moved D65 178.5 mm to (214.2, 56.9)
- moved D73 170.0 mm to (248.3, 31.5)
- moved D74 170.0 mm to (251.5, 31.5)
- moved D76 170.0 mm to (257.8, 31.5)
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Routing:
- net Net-(D81-A): track 0.00 -> 134.4 mm
- net Net-(D79-A): track 0.00 -> 129.0 mm
- net Net-(D80-A): track 0.00 -> 128.9 mm
- net Net-(D72-A): track 0.00 -> 117.6 mm
- net Net-(D70-A): track 0.01 -> 116.9 mm
- net Net-(D71-A): track 0.01 -> 116.8 mm
- net Net-(D69-A): track 0.01 -> 116.3 mm
- net Net-(D68-A): track 0.01 -> 114.4 mm
- net Net-(D66-A): track 1.36 -> 115.5 mm
- net Net-(D67-A): track 0.01 -> 113.5 mm
- net Net-(D65-A): track 0.01 -> 111.6 mm
- net Net-(D59-A): track 0.00 -> 91.6 mm
- net Net-(D58-A): track 0.00 -> 91.6 mm
- net Net-(D57-A): track 0.00 -> 91.6 mm
- net Net-(D53-A): track 0.00 -> 87.3 mm
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
Commit message: should work
Parts:
- C3, C4, C5, C6: footprint Capacitor_THT:C_Radial_D10.0mm_H12.5mm_P5.00mm -> Capacitor_THT:C_Radial_D4.0mm_H7.0mm_P1.50mm
- J3: moved to F.Cu
- moved SW90 313.8 mm to (211.3, 88.2), turned to 90 degrees
- moved D86 277.4 mm to (490.4, 56.9)
- moved D88 277.3 mm to (528.5, 56.9)
- moved D85 271.9 mm to (463.9, 56.9)
- moved D87 263.5 mm to (511.5, 56.9)
- moved D50 259.1 mm to (526.4, 56.9)
- moved D33 258.6 mm to (524.3, 56.9)
- moved D16 258.5 mm to (522.2, 56.9)
- moved D77 249.8 mm to (509.4, 56.9)
- moved C2 245.8 mm to (109.7, 120.5), turned to 180 degrees
- moved D49 243.4 mm to (507.3, 56.9)
- moved D15 243.0 mm to (503.1, 56.9)
- moved D32 243.0 mm to (505.2, 56.9)
- moved D84 239.5 mm to (444.9, 56.9)
- moved D48 227.8 mm to (488.3, 56.9)
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Connections:
- J2 pad 6: Net-(J2-Pin_6) -> unconnected-(J2-Pin_6-Pad6)
- R1 pad 2: Net-(J2-Pin_6) -> Net-(J1-Pin_1)
Routing:
- net Row 2: track 2.34 -> 618.4 mm
- net Row 1: track 0.00 -> 612.9 mm
- net Row 5: track 0.00 -> 586.0 mm
- net Row 0: track 0.00 -> 580.4 mm
- net Row 4: track 7.16 -> 539.4 mm
- net Row 3: track 0.01 -> 489.2 mm
- net Column 16: track 104.8 -> 478.4 mm
- net Column 15: track 107.3 -> 466.5 mm
- net Column 14: track 104.8 -> 442.6 mm
- net Column 13: track 123.5 -> 427.6 mm
- net Column 12: track 121.6 -> 406.4 mm
- net Column 11: track 123.5 -> 399.7 mm
- net Column 10: track 123.5 -> 367.2 mm
- net Column 9: track 99.5 -> 332.3 mm
- net Column 7: track 99.5 -> 321.3 mm
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- added copper zone on B.Cu, net GND
- added copper zone on F.Cu, net GND
Other:
- board outline added: 440.5 x 147.4 mm

Commit message: should work
Parts:
- added REF**: MountingHole_3.2mm_M3, MountingHole:MountingHole_3.2mm_M3, F.Cu at (331.6, 254.3)
- added REF**: MountingHole_3.2mm_M3, MountingHole:MountingHole_3.2mm_M3, F.Cu at (156.6, 129.3)
- added REF**: MountingHole_3.2mm_M3, MountingHole:MountingHole_3.2mm_M3, F.Cu at (286.6, 164.3)
- added REF**: MountingHole_3.2mm_M3, MountingHole:MountingHole_3.2mm_M3, F.Cu at (91.6, 254.3)
- added REF**: MountingHole_3.2mm_M3, MountingHole:MountingHole_3.2mm_M3, F.Cu at (461.6, 214.3)
- added REF**: MountingHole_3.2mm_M3, MountingHole:MountingHole_3.2mm_M3, F.Cu at (266.6, 254.3)
- added REF**: MountingHole_3.2mm_M3, MountingHole:MountingHole_3.2mm_M3, F.Cu at (511.6, 239.3)
- added REF**: MountingHole_3.2mm_M3, MountingHole:MountingHole_3.2mm_M3, F.Cu at (156.6, 254.3)
- added REF**: MountingHole_3.2mm_M3, MountingHole:MountingHole_3.2mm_M3, F.Cu at (516.6, 129.3)
- added REF**: MountingHole_3.2mm_M3, MountingHole:MountingHole_3.2mm_M3, F.Cu at (461.6, 239.3)
- added REF**: MountingHole_3.2mm_M3, MountingHole:MountingHole_3.2mm_M3, F.Cu at (161.6, 209.3)
- added REF**: MountingHole_3.2mm_M3, MountingHole:MountingHole_3.2mm_M3, F.Cu at (91.6, 129.3)
- added REF**: MountingHole_3.2mm_M3, MountingHole:MountingHole_3.2mm_M3, F.Cu at (511.6, 214.3)
- added REF**: MountingHole_3.2mm_M3, MountingHole:MountingHole_3.2mm_M3, F.Cu at (366.6, 164.3)
- moved D16 70.9 mm to (504.2, 125.5)
- moved D29 70.9 mm to (420.6, 125.5)
- moved D31 70.9 mm to (468.2, 125.5)
- moved D33 70.9 mm to (506.3, 125.5)
- moved D76 70.9 mm to (443.8, 125.5)
- moved D77 70.9 mm to (491.4, 125.5)
- moved R1 70.9 mm to (107.5, 255.0)
- moved SW10 70.9 mm to (388.9, 144.4)
- moved SW16 70.9 mm to (512.7, 144.4)
- moved SW42 70.9 mm to (341.2, 192.0)
- moved SW50 70.9 mm to (512.7, 192.0)
- moved SW54 70.9 mm to (250.8, 211.0)
- moved SW55 70.9 mm to (269.8, 211.0)
- moved SW60 70.9 mm to (365.1, 211.0)
- moved SW8 70.9 mm to (341.2, 144.4)
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