File: pcb/orione-v2/orione-v2.kicad_pcb (KiCad board)
At the start: 2 copper layers, 318.9 x 119.5 mm, 133 parts, among them SW1 SW_Push, SW10 SW_Push, SW11 SW_Push, SW12 SW_Push, SW13 SW_Push, SW14 SW_Push, SW15 SW_Push, SW16 SW_Push, SW17 SW_Push, SW18 SW_Push, SW19 SW_Push, SW2 SW_Push, SW20 SW_Push, SW21 SW_Push, SW22 SW_Push, SW23 SW_Push, SW24 SW_Push, SW25 SW_Push, SW26 SW_Push, SW27 SW_Push, SW28 SW_Push, SW29 SW_Push, SW3 SW_Push, SW30 SW_Push, SW31 SW_Push, SW32 SW_Push, SW33 SW_Push, SW34 SW_Push, SW35 SW_Push, SW36 SW_Push, SW37 SW_Push, SW38 SW_Push, SW39 SW_Push, SW4 SW_Push, SW40 SW_Push, SW41 SW_Push, SW42 SW_Push, SW43 SW_Push, SW44 SW_Push, SW45 SW_Push, SW46 SW_Push, SW47 SW_Push, SW48 SW_Push, SW49 SW_Push, SW5 SW_Push, SW50 SW_Push, SW51 SW_Push, SW52 SW_Push, SW53 SW_Push, SW54 SW_Push, SW55 SW_Push, SW56 SW_Push, SW57 SW_Push, SW58 SW_Push, SW59 SW_Push, SW6 SW_Push, SW60 SW_Push, SW61 SW_Push, SW62 SW_Push, SW63 RotaryEncoder_Switch, SW7 SW_Push, SW8 SW_Push, SW9 SW_Push

Commit message: pcb
Parts:
- removed SW63: RotaryEncoder_Switch, Rotary_Encoder:RotaryEncoder_Alps_EC11E-Switch_Vertical_H20mm
- added J1: Conn_01x05_Socket, Connector_PinSocket_2.54mm:PinSocket_1x05_P2.54mm_Vertical, F.Cu at (55.9, 161.0)
- moved D63 8.04 mm to (59.7, 171.5)
- moved A1 1.10 mm to (61.0, 102.8)
- moved D55 0.09 mm to (108.8, 92.5)
- moved D30 0.08 mm to (103.9, 86.1)
- moved D16 0.08 mm to (101.4, 82.9)
- moved D43 0.08 mm to (106.4, 89.3)
- moved D62 0.08 mm to (339.5, 92.5)
- moved D53 0.06 mm to (337.0, 89.3)
Connections:
- A1 pad 25: Net-(A1-GPIO19) -> Rotary_clk
- A1 pad 26: Net-(A1-GPIO20) -> Rotary_dt
- A1 pad 27: Net-(A1-GPIO21) -> Rotary_sw
- A1 pad 36: unconnected-(A1-3V3-Pad36) -> Power
- D1 pad 1: Row 0 -> Column 0
- D10 pad 1: Row 0 -> Column 9
- D11 pad 1: Row 0 -> Column 10
- D12 pad 1: Row 0 -> Column 11
- D13 pad 1: Row 0 -> Column 12
- D14 pad 1: Row 0 -> Column 13
- D15 pad 1: Row 1 -> Column 0
- D16 pad 1: Row 1 -> Column 1
- D17 pad 1: Row 1 -> Column 2
- D18 pad 1: Row 1 -> Column 3
- D19 pad 1: Row 1 -> Column 4
- D2 pad 1: Row 0 -> Column 1
- D20 pad 1: Row 1 -> Column 5
- D21 pad 1: Row 1 -> Column 6
- D22 pad 1: Row 1 -> Column 7
- D23 pad 1: Row 1 -> Column 8
- D24 pad 1: Row 1 -> Column 9
- D25 pad 1: Row 1 -> Column 10
- D26 pad 1: Row 1 -> Column 11
- D27 pad 1: Row 1 -> Column 12
- D28 pad 1: Row 1 -> Column 13
- D29 pad 1: Row 2 -> Column 0
- D3 pad 1: Row 0 -> Column 2
- D30 pad 1: Row 2 -> Column 1
- D31 pad 1: Row 2 -> Column 2
- D32 pad 1: Row 2 -> Column 3
- D33 pad 1: Row 2 -> Column 4
- D34 pad 1: Row 2 -> Column 5
- D35 pad 1: Row 2 -> Column 6
- D36 pad 1: Row 2 -> Column 7
- D37 pad 1: Row 2 -> Column 8
- D38 pad 1: Row 2 -> Column 9
- D39 pad 1: Row 2 -> Column 10
- D4 pad 1: Row 0 -> Column 3
- D40 pad 1: Row 2 -> Column 11
- D41 pad 1: Row 2 -> Column 13
- D42 pad 1: Row 3 -> Column 0
- D43 pad 1: Row 3 -> Column 1
- D44 pad 1: Row 3 -> Column 2
- D45 pad 1: Row 3 -> Column 3
- D46 pad 1: Row 3 -> Column 4
- D47 pad 1: Row 3 -> Column 5
- D48 pad 1: Row 3 -> Column 6
- D49 pad 1: Row 3 -> Column 7
- D5 pad 1: Row 0 -> Column 4
- D50 pad 1: Row 3 -> Column 8
- D51 pad 1: Row 3 -> Column 9
- D52 pad 1: Row 3 -> Column 10
- D53 pad 1: Row 3 -> Column 13
- D54 pad 1: Row 4 -> Column 0
- D55 pad 1: Row 4 -> Column 1
- D56 pad 1: Row 4 -> Column 2
- D57 pad 1: Row 4 -> Column 5
- D58 pad 1: Row 4 -> Column 9
- D59 pad 1: Row 4 -> Column 10
- D6 pad 1: Row 0 -> Column 5
- D60 pad 1: Row 4 -> Column 11
- D61 pad 1: Row 4 -> Column 12
- D62 pad 1: Row 4 -> Column 13
- D7 pad 1: Row 0 -> Column 6
- D8 pad 1: Row 0 -> Column 7
- D9 pad 1: Row 0 -> Column 8
- SW1 pad 1: Net-(D1-A) -> Row 0
- SW1 pad 2: Column 0 -> Net-(D1-A)
- SW10 pad 1: Net-(D10-A) -> Row 0
- SW10 pad 2: Column 9 -> Net-(D10-A)
- SW11 pad 1: Net-(D11-A) -> Row 0
- SW11 pad 2: Column 10 -> Net-(D11-A)
- SW12 pad 1: Net-(D12-A) -> Row 0
- SW12 pad 2: Column 11 -> Net-(D12-A)
- SW13 pad 1: Net-(D13-A) -> Row 0
- SW13 pad 2: Column 12 -> Net-(D13-A)
- SW14 pad 1: Net-(D14-A) -> Row 0
- SW14 pad 2: Column 13 -> Net-(D14-A)
- SW15 pad 1: Net-(D15-A) -> Row 1
- SW15 pad 2: Column 0 -> Net-(D15-A)
- SW16 pad 1: Net-(D16-A) -> Row 1
- SW16 pad 2: Column 1 -> Net-(D16-A)
- SW17 pad 1: Net-(D17-A) -> Row 1
- SW17 pad 2: Column 2 -> Net-(D17-A)
- SW18 pad 1: Net-(D18-A) -> Row 1
- SW18 pad 2: Column 3 -> Net-(D18-A)
- SW19 pad 1: Net-(D19-A) -> Row 1
- SW19 pad 2: Column 4 -> Net-(D19-A)
- SW2 pad 1: Net-(D2-A) -> Row 0
- SW2 pad 2: Column 1 -> Net-(D2-A)
- SW20 pad 1: Net-(D20-A) -> Row 1
- SW20 pad 2: Column 5 -> Net-(D20-A)
- SW21 pad 1: Net-(D21-A) -> Row 1
- SW21 pad 2: Column 6 -> Net-(D21-A)
- SW22 pad 1: Net-(D22-A) -> Row 1
- SW22 pad 2: Column 7 -> Net-(D22-A)
- SW23 pad 1: Net-(D23-A) -> Row 1
- SW23 pad 2: Column 8 -> Net-(D23-A)
- SW24 pad 1: Net-(D24-A) -> Row 1
- SW24 pad 2: Column 9 -> Net-(D24-A)
- SW25 pad 1: Net-(D25-A) -> Row 1
- SW25 pad 2: Column 10 -> Net-(D25-A)
- SW26 pad 1: Net-(D26-A) -> Row 1
- SW26 pad 2: Column 11 -> Net-(D26-A)
- SW27 pad 1: Net-(D27-A) -> Row 1
- SW27 pad 2: Column 12 -> Net-(D27-A)
- SW28 pad 1: Net-(D28-A) -> Row 1
- SW28 pad 2: Column 13 -> Net-(D28-A)
- SW29 pad 1: Net-(D29-A) -> Row 2
- SW29 pad 2: Column 0 -> Net-(D29-A)
- SW3 pad 1: Net-(D3-A) -> Row 0
- SW3 pad 2: Column 2 -> Net-(D3-A)
- SW30 pad 1: Net-(D30-A) -> Row 2
- SW30 pad 2: Column 1 -> Net-(D30-A)
- SW31 pad 1: Net-(D31-A) -> Row 2
- SW31 pad 2: Column 2 -> Net-(D31-A)
- SW32 pad 1: Net-(D32-A) -> Row 2
- SW32 pad 2: Column 3 -> Net-(D32-A)
- SW33 pad 1: Net-(D33-A) -> Row 2
- SW33 pad 2: Column 4 -> Net-(D33-A)
- SW34 pad 1: Net-(D34-A) -> Row 2
- SW34 pad 2: Column 5 -> Net-(D34-A)
- SW35 pad 1: Net-(D35-A) -> Row 2
- SW35 pad 2: Column 6 -> Net-(D35-A)
- SW36 pad 1: Net-(D36-A) -> Row 2
- SW36 pad 2: Column 7 -> Net-(D36-A)
- SW37 pad 1: Net-(D37-A) -> Row 2
- SW37 pad 2: Column 8 -> Net-(D37-A)
- SW38 pad 1: Net-(D38-A) -> Row 2
- SW38 pad 2: Column 9 -> Net-(D38-A)
- SW39 pad 1: Net-(D39-A) -> Row 2
- SW39 pad 2: Column 10 -> Net-(D39-A)
- SW4 pad 1: Net-(D4-A) -> Row 0
- SW4 pad 2: Column 3 -> Net-(D4-A)
- SW40 pad 1: Net-(D40-A) -> Row 2
- SW40 pad 2: Column 11 -> Net-(D40-A)
- SW41 pad 1: Net-(D41-A) -> Row 2
- SW41 pad 2: Column 13 -> Net-(D41-A)
- SW42 pad 1: Net-(D42-A) -> Row 3
- SW42 pad 2: Column 0 -> Net-(D42-A)
- SW43 pad 1: Net-(D43-A) -> Row 3
- SW43 pad 2: Column 1 -> Net-(D43-A)
- SW44 pad 1: Net-(D44-A) -> Row 3
- SW44 pad 2: Column 2 -> Net-(D44-A)
- SW45 pad 1: Net-(D45-A) -> Row 3
- SW45 pad 2: Column 3 -> Net-(D45-A)
- SW46 pad 1: Net-(D46-A) -> Row 3
- SW46 pad 2: Column 4 -> Net-(D46-A)
- SW47 pad 1: Net-(D47-A) -> Row 3
- SW47 pad 2: Column 5 -> Net-(D47-A)
- SW48 pad 1: Net-(D48-A) -> Row 3
- SW48 pad 2: Column 6 -> Net-(D48-A)
- SW49 pad 1: Net-(D49-A) -> Row 3
- SW49 pad 2: Column 7 -> Net-(D49-A)
- SW5 pad 1: Net-(D5-A) -> Row 0
- SW5 pad 2: Column 4 -> Net-(D5-A)
- SW50 pad 1: Net-(D50-A) -> Row 3
- SW50 pad 2: Column 8 -> Net-(D50-A)
- SW51 pad 1: Net-(D51-A) -> Row 3
- SW51 pad 2: Column 9 -> Net-(D51-A)
- SW52 pad 1: Net-(D52-A) -> Row 3
- SW52 pad 2: Column 10 -> Net-(D52-A)
- SW53 pad 1: Net-(D53-A) -> Row 3
- SW53 pad 2: Column 13 -> Net-(D53-A)
- SW54 pad 1: Net-(D54-A) -> Row 4
- SW54 pad 2: Column 0 -> Net-(D54-A)
- SW55 pad 1: Net-(D55-A) -> Row 4
- SW55 pad 2: Column 1 -> Net-(D55-A)
- SW56 pad 1: Net-(D56-A) -> Row 4
- SW56 pad 2: Column 2 -> Net-(D56-A)
- SW57 pad 1: Net-(D57-A) -> Row 4
- SW57 pad 2: Column 5 -> Net-(D57-A)
- SW58 pad 1: Net-(D58-A) -> Row 4
- SW58 pad 2: Column 9 -> Net-(D58-A)
- SW59 pad 1: Net-(D59-A) -> Row 4
- SW59 pad 2: Column 10 -> Net-(D59-A)
- SW6 pad 1: Net-(D6-A) -> Row 0
- SW6 pad 2: Column 5 -> Net-(D6-A)
- SW60 pad 1: Net-(D60-A) -> Row 4
- SW60 pad 2: Column 11 -> Net-(D60-A)
- SW61 pad 1: Net-(D61-A) -> Row 4
- SW61 pad 2: Column 12 -> Net-(D61-A)
- SW62 pad 1: Net-(D62-A) -> Row 4
- SW62 pad 2: Column 13 -> Net-(D62-A)
- SW7 pad 1: Net-(D7-A) -> Row 0
- SW7 pad 2: Column 6 -> Net-(D7-A)
- SW8 pad 1: Net-(D8-A) -> Row 0
- SW8 pad 2: Column 7 -> Net-(D8-A)
- SW9 pad 1: Net-(D9-A) -> Row 0
- SW9 pad 2: Column 8 -> Net-(D9-A)
Routing:
- net Row 0: track 291.5 -> 398.3 mm, vias 0 -> 1
- net Row 1: track 294.1 -> 398.4 mm, vias 0 -> 1
- net Row 4: track 295.8 -> 385.6 mm, vias 0 -> 1
- net Power: track 0.00 -> 79.5 mm
- net Column 1: track 149.4 -> 75.2 mm
- net Column 13: track 370.4 -> 299.2 mm, vias 1 -> 0
- net Column 2: track 165.5 -> 94.5 mm
- net Column 9: track 305.2 -> 239.4 mm
- net Column 0: track 120.0 -> 54.4 mm
- net Column 10: track 323.5 -> 261.4 mm
- net Column 5: track 217.8 -> 157.9 mm
- net Row 2: track 295.5 -> 355.1 mm, vias 0 -> 1
- net Column 12: track 344.9 -> 286.8 mm, vias 1 -> 0
- net Column 7: track 248.5 -> 192.7 mm
- net Rotary_dt: track 0.00 -> 55.5 mm
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Other:
- board size 318.9 x 119.5 mm -> 319.9 x 119.6 mm
- board text added: "D17"
- board text added: "Orione 2.0 by ilBuso"
- board text removed: "DUCK 1.0 by ilBuso"
