File: pcb/orione-v2/orione-v2.kicad_sch (KiCad schematic)
At the start: 3 parts, among them SW63 RotaryEncoder_Switch

Commit message: pcb
Parts:
- removed SW63: RotaryEncoder_Switch, Rotary_Encoder:RotaryEncoder_Alps_EC11E-Switch_Vertical_H20mm, symbol Device:RotaryEncoder_Switch
- added J1: Conn_01x05_Socket, Connector_PinSocket_2.54mm:PinSocket_1x05_P2.54mm_Vertical, symbol Connector:Conn_01x05_Socket
Connections:
- net GND: now also J1.1 (Pin_1)
- net Rotary_clk: now reaches A1.25 (GPIO19)
- net Rotary_clk: now also J1.5 (Pin_5)
- net Rotary_dt: now reaches A1.26 (GPIO20)
- net Rotary_dt: now also J1.4 (Pin_4)
- net Rotary_sw: now reaches A1.27 (GPIO21)
- net Rotary_sw: now also J1.3 (Pin_3)
- net Power: now reaches A1.36 (3V3)
- net Power: now also J1.2 (Pin_2)
- no-connect marks 8 -> 9
